File: 6502-ACE.kicad_sch (KiCad schematic)
At the start: 156 parts, among them J10 RESET SW, J11 6502 CART, J12 6502 BUS, J13 PADDLES, J14 AUDIO L, J15 AUDIO R, J16 Compact Flash, J17 DB9 MALE (DTE), J18 CTS EN, J19 DCD EN, J2 PHI2 Select, J20 ACT LED, J21 IDE, J3 PS/2, J4 JOYSTICK A, J5 JOYSTICK B, J6 PORT B, J7 PORT B, J8 PORT A, J9 PORT A, SW1 `, SW10 1, SW11 9, SW12 W, SW13 P, SW14 D, SW15 ', SW16 B, SW17 MENU, SW18 2, SW19 0, SW2 8, SW20 E, SW21 [, SW22 F, SW23 ENTER, SW24 N, SW25 ALT, SW26 R ALT, SW27 3, SW28 -, SW29 R, SW3 Q, SW30 ], SW31 G, SW32 DELETE, SW33 M, SW34 SPACE, SW35 4, SW36 =, SW37 T, SW38 \, SW39 H, SW4 O, SW40 SHIFT, SW41 R SHIFT, SW42 ,, SW43 FN, SW44 5, SW45 BACKSPACE, SW46 Y, SW47 INSERT, SW48 J, SW49 Z, SW5 S, SW50 ., SW51 LEFT ARROW, SW52 6, SW53 ESCAPE, SW54 U, SW55 CAPS LOCK, SW56 K, SW57 X, SW58 /, SW59 DOWN ARROW, SW6 ;, SW60 7, SW61 TAB, SW62 I, SW63 A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

Commit message: Update PDF
Parts:
- added unit 1 of U1
- added unit 5 of U14
- added unit 2 of U15
- added unit 5 of U16
- added unit 1 of U5
- added unit 1 of U6
Connections:
- net A14: now also U1.1, U1.2, U6.2; no longer U1.1, U1.2, U6.2
- net GND: now also U14.7 (GND), U15.7 (GND), U16.7 (GND); no longer U14.7 (GND), U15.7 (GND), U16.7 (GND)
- net HRDB: now also U6.1; no longer U6.1
- net REB: now also U5.3; no longer U5.3
- net VCC: now also U14.14 (VCC), U15.14 (VCC), U16.14 (VCC); no longer U14.14 (VCC), U15.14 (VCC), U16.14 (VCC)
- net at U1.4: now also U1.3; no longer U1.3
- net at U6.4, U6.5: now also U6.3; no longer U6.3
- new net: U5.1, U5.2, U6.11
Other:
- moved on the sheet: D1, J16, J20, J21, R26, R27, R28, R29, R30, R31

Commit message: Finish Schematic
Parts:
- removed D1: ACT, LED_SMD:LED_0805_2012Metric, symbol Device:LED
- removed J16: Compact Flash, symbol 6502-ACE:Compact Flash
- removed J20: ACT LED, Connector_JST:JST_XH_B2B-XH-A_1x02_P2.50mm_Vertical, symbol Connector_Generic:Conn_01x02
- removed J21: IDE, symbol Connector_Generic:Conn_02x22_Odd_Even
- removed R26, R27, R28, R29: 1k, Resistor_SMD:R_0805_2012Metric, symbol Device:R
- removed R30, R31: 330, Resistor_SMD:R_0805_2012Metric, symbol Device:R
- added C10, C11, C12, C13, C14, C15, C16, C17, C18, C19, C20, C21, C22, C23, C24, C25, C26, C27, C28, C29, C30, C9: 100nF, Capacitor_THT:C_Disc_D5.0mm_W2.5mm_P2.50mm, symbol Device:C
- added D3: POWER LED, LED_THT:LED_D3.0mm, symbol Device:LED
- added J10: AUDIO, Connector_JST:JST_XH_B2B-XH-A_1x02_P2.50mm_Vertical, symbol Connector_Generic:Conn_01x02
- added J16: STORAGE, Connector_PinHeader_2.54mm:PinHeader_2x10_P2.54mm_Vertical, symbol Connector_Generic:Conn_02x10_Odd_Even
- added J20: 5V DC, Connector_BarrelJack:BarrelJack_Horizontal, symbol Connector:Barrel_Jack_Switch
- added J21: VCC, Connector_JST:JST_XH_B2B-XH-A_1x02_P2.50mm_Vertical, symbol Connector_Generic:Conn_01x02
- added J22: POWER LED, Connector_JST:JST_XH_B2B-XH-A_1x02_P2.50mm_Vertical, symbol Connector_Generic:Conn_01x02
- added R10, R12, R13, R14, R15, R4, R6, R8: 1K, Resistor_THT:R_Axial_DIN0204_L3.6mm_D1.6mm_P5.08mm_Horizontal, symbol Device:R
- added R36: 330, Resistor_THT:R_Axial_DIN0204_L3.6mm_D1.6mm_P5.08mm_Horizontal, symbol Device:R
- added SW1: IO ENABLE, Button_Switch_THT:SW_DIP_SPSTx08_Slide_9.78x22.5mm_W7.62mm_P2.54mm, symbol Switch:SW_DIP_x08
- added SW11: POWER, 6502-ACE:SW_400MSP1R6BLKM6QE, symbol Switch:SW_SPDT
- added TP1: GND, TestPoint:TestPoint_Pad_2.5x2.5mm, symbol Connector:TestPoint
- added TP2: VCC, TestPoint:TestPoint_Pad_2.5x2.5mm, symbol Connector:TestPoint
- BT1: Availability In Stock -> (none); Check_prices https://www.snapeda.com/parts/BAT-HLD-001-THM/Linx+Technolo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 -> (none); Description_1 Holder for CR2032 and CR2025 Batteries, Through-Hole Mount,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 -> (none); Digikey (none) -> BAT-HLD-001-THM-ND; MF Linx Technologies -> (none); MP BAT-HLD-001-THM -> (none); MPN (none) -> BAT-HLD-001-THM; Mouser (none) -> 712-BAT-HLD-001-THM; Package None -> (none); Price None -> (none); Purchase-URL https://www.snapeda.com/api/url_track_click_mouser/?unipart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 -> (none); SnapEDA_Link https://www.snapeda.com/parts/BAT-HLD-001-THM/Linx+Technolo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 -> (none)
- C1: footprint Capacitor_SMD:C_0805_2012Metric -> Capacitor_THT:C_Disc_D5.0mm_W2.5mm_P2.50mm; LCSC C49678 -> (none)
- C2, C5, C6, C7, C8: footprint Capacitor_SMD:C_0805_2012Metric -> Capacitor_THT:C_Disc_D5.0mm_W2.5mm_P2.50mm; LCSC C28323 -> (none)
- C3, C4: footprint Capacitor_SMD:C_0805_2012Metric -> Capacitor_THT:C_Disc_D5.0mm_W2.5mm_P2.50mm; LCSC C28260 -> (none)
- D1: renamed from D2; Amazon (none) -> https://www.amazon.com/gp/product/B0CKSNPVH8; Digikey (none) -> BAT85SCT-ND; Mouser (none) -> 78-BAT85S; now in the parts list
- D2: renamed from D3; Amazon (none) -> https://www.amazon.com/gp/product/B0CKSNPVH8; Digikey (none) -> BAT85SCT-ND; Mouser (none) -> 78-BAT85S; now in the parts list
- J1: renamed from J2; now in the parts list
- J12: renamed from J14; Digikey https://www.digikey.com/en/products/detail/switchcraft-inc/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 -> PJRAN1X1U02X-ND; Mouser (none) -> 502-PJRAN1X1U02X
- J13: renamed from J15; Digikey https://www.digikey.com/en/products/detail/switchcraft-inc/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 -> PJRAN1X1U03X-ND; Mouser (none) -> 502-PJRAN1X1U03X
- J14: renamed from J11; value 6502 CART -> CART; Digikey (none) -> A31723-ND; Mouser (none) -> 571-5-5530843-4; now in the parts list
- J15: renamed from J12; value 6502 BUS -> BUS; now in the parts list
- J17: Mouser (none) -> 649-D09P33E4GX00LF
- J18, J19: now in the parts list
- J2: renamed from J3; Amazon (none) -> https://www.amazon.com/dp/B08GS3QL7T
- J3: renamed from J4; Mouser (none) -> 649-D09P33E4GX00LF; now in the parts list
- J4: renamed from J5; Mouser (none) -> 649-D09P33E4GX00LF; now in the parts list
- J5: renamed from J6; now in the parts list
- J6: renamed from J7; now in the parts list
- J7: renamed from J8; now in the parts list
- J8: renamed from J9; now in the parts list
- J9: renamed from J10; now in the parts list
- R1, R2, R3, R32: footprint Resistor_SMD:R_0805_2012Metric -> Resistor_THT:R_Axial_DIN0204_L3.6mm_D1.6mm_P5.08mm_Horizontal; LCSC C17513 -> (none)
- R11: renamed from R33; footprint Resistor_SMD:R_0805_2012Metric -> Resistor_THT:R_Axial_DIN0204_L3.6mm_D1.6mm_P5.08mm_Horizontal; LCSC C17513 -> (none)
- R16: renamed from R7; now in the parts list
- R17: renamed from R8; now in the parts list
- R18: renamed from R9; now in the parts list
- R19: renamed from R10; now in the parts list
- R20: renamed from R11; now in the parts list
- R21: renamed from R12; now in the parts list
- R22: renamed from R13; now in the parts list
- R23: renamed from R14; now in the parts list
- R24: renamed from R15; now in the parts list
- R25: renamed from R16; now in the parts list
- R26: renamed from R17; now in the parts list
- R27: renamed from R18; now in the parts list
- R28: renamed from R19; now in the parts list
- R29: renamed from R20; now in the parts list
- R30: renamed from R21; now in the parts list
- R31: renamed from R22; now in the parts list
- R33: renamed from R23; footprint Resistor_SMD:R_0805_2012Metric -> Resistor_THT:R_Axial_DIN0204_L3.6mm_D1.6mm_P5.08mm_Horizontal; LCSC C17513 -> (none)
- R34: renamed from R24; footprint Resistor_SMD:R_0805_2012Metric -> Resistor_THT:R_Axial_DIN0204_L3.6mm_D1.6mm_P5.08mm_Horizontal; LCSC C17513 -> (none)
- R35: renamed from R25; footprint Resistor_SMD:R_0805_2012Metric -> Resistor_THT:R_Axial_DIN0204_L3.6mm_D1.6mm_P5.08mm_Horizontal; LCSC C17513 -> (none)
- R5: renamed from R4; footprint Resistor_SMD:R_0805_2012Metric -> Resistor_THT:R_Axial_DIN0204_L3.6mm_D1.6mm_P5.08mm_Horizontal; LCSC C17513 -> (none)
- R7: renamed from R5; footprint Resistor_SMD:R_0805_2012Metric -> Resistor_THT:R_Axial_DIN0204_L3.6mm_D1.6mm_P5.08mm_Horizontal; LCSC C17513 -> (none)
- R9: renamed from R6; footprint Resistor_SMD:R_0805_2012Metric -> Resistor_THT:R_Axial_DIN0204_L3.6mm_D1.6mm_P5.08mm_Horizontal; LCSC C17513 -> (none)
- SW10: renamed from SW9; now in the parts list
- SW12: renamed from SW10; now in the parts list
- SW13: renamed from SW11; now in the parts list
- SW14: renamed from SW12; now in the parts list
- SW15: renamed from SW13; now in the parts list
- SW16: renamed from SW14; now in the parts list
- SW17: renamed from SW15; now in the parts list
- SW18: renamed from SW16; now in the parts list
- SW19: renamed from SW17; now in the parts list
- SW2: renamed from SW1; now in the parts list
- SW20: renamed from SW18; now in the parts list
- SW21: renamed from SW19; now in the parts list
- SW22: renamed from SW20; now in the parts list
- SW23: renamed from SW21; now in the parts list
- SW24: renamed from SW22; now in the parts list
- SW25: renamed from SW23; now in the parts list
- SW26: renamed from SW24; now in the parts list
- SW27: renamed from SW25; now in the parts list
- SW28: renamed from SW26; now in the parts list
- SW29: renamed from SW27; now in the parts list
- SW3: renamed from SW2; now in the parts list
- SW30: renamed from SW28; now in the parts list
- SW31: renamed from SW29; now in the parts list
- SW32: renamed from SW30; now in the parts list
- SW33: renamed from SW31; now in the parts list
- SW34: renamed from SW32; now in the parts list
- SW35: renamed from SW33; now in the parts list
- SW36: renamed from SW34; now in the parts list
- SW37: renamed from SW35; now in the parts list
- SW38: renamed from SW36; now in the parts list
- SW39: renamed from SW37; now in the parts list
- SW4: renamed from SW3; now in the parts list
- SW40: renamed from SW38; now in the parts list
- SW41: renamed from SW39; now in the parts list
- SW42: renamed from SW40; now in the parts list
- SW43: renamed from SW41; now in the parts list
- SW44: renamed from SW42; now in the parts list
- SW45: renamed from SW43; now in the parts list
- SW46: renamed from SW44; now in the parts list
- SW47: renamed from SW45; now in the parts list
- SW48: renamed from SW46; now in the parts list
- SW49: renamed from SW47; now in the parts list
- SW5: renamed from SW4; now in the parts list
- SW50: renamed from SW48; now in the parts list
- SW51: renamed from SW49; now in the parts list
- SW52: renamed from SW50; now in the parts list
- SW53: renamed from SW51; now in the parts list
- SW54: renamed from SW52; now in the parts list
- SW55: renamed from SW53; now in the parts list
- SW56: renamed from SW54; now in the parts list
- SW57: renamed from SW55; now in the parts list
- SW58: renamed from SW56; now in the parts list
- SW59: renamed from SW57; now in the parts list
- SW6: renamed from SW5; now in the parts list
- SW60: renamed from SW58; now in the parts list
- SW61: renamed from SW59; now in the parts list
- SW62: renamed from SW60; now in the parts list
- SW63: renamed from SW61; now in the parts list
- SW64: renamed from SW62; now in the parts list
- SW65: renamed from SW63; now in the parts list
- SW66: renamed from SW64; now in the parts list
- SW67: renamed from SW65; now in the parts list
- SW68: renamed from SW66; now in the parts list
- SW69: renamed from SW67; now in the parts list
- SW7: renamed from SW6; now in the parts list
- SW8: renamed from SW7; now in the parts list
- SW9: renamed from SW8; now in the parts list
- U1, U14, U16, U6: footprint Package_SO:SOIC-14_3.9x8.7mm_P1.27mm -> Package_DIP:DIP-14_W7.62mm_Socket_LongPads; Digikey (none) -> 296-1563-5-ND; LCSC C5586 -> (none); Mouser (none) -> 595-SN74HC00N
- U10: Digikey (none) -> 1450-1027-ND; Mouser (none) -> 913-AS6C4008-55PCN
- U11: renamed from U12; Mouser (none) -> 955-W65C22N6TPG-14
- U12: renamed from U11; footprint Package_SO:SOIC-20W_7.5x12.8mm_P1.27mm -> Package_DIP:DIP-20_W7.62mm_Socket_LongPads; Digikey (none) -> 296-12815-5-ND; LCSC C5608 -> (none); Mouser (none) -> 595-CD74HC573EE4
- U13: footprint Package_SO:SOIC-20W_7.5x12.8mm_P1.27mm -> Package_DIP:DIP-20_W7.62mm_Socket_LongPads; Digikey (none) -> 296-12815-5-ND; LCSC C5608 -> (none); Mouser (none) -> 595-CD74HC573EE4
- U15: footprint Package_SO:SOIC-14_3.9x8.7mm_P1.27mm -> Package_DIP:DIP-14_W7.62mm_Socket_LongPads; Digikey (none) -> 296-9196-5-ND; LCSC C19818870 -> (none); Mouser (none) -> 595-CD74HC30E
- U17: Digikey (none) -> ATMEGA1284-PU-ND; Mouser (none) -> 556-ATMEGA1284-PU; now in the parts list
- U18: Mouser (none) -> 700-DS1511Y; now in the parts list
- U19: Availability Not in stock -> (none); Check_prices https://www.snapeda.com/parts/AY-3-8912/General+Instrument/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 -> (none); Description_1 (none) -> (none); MANUFACTURER ST Microelectronics -> (none); MF General Instrument -> (none); MP AY-3-8912 -> (none); Package None -> (none); Price None -> (none); SnapEDA_Link https://www.snapeda.com/parts/AY-3-8912/General+Instrument/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 -> (none)
- U2: Mouser (none) -> 955-W65C02S6TPG-14
- U22: Digikey (none) -> MAX238CNG+-ND; Mouser (none) -> 700-MAX238CNG
- U3: Digikey (none) -> 1450-1033-ND; Mouser (none) -> 913-AS6C62256-55PCN
- U4: renamed from U5; footprint Package_SO:SOIC-14_3.9x8.7mm_P1.27mm -> Package_DIP:DIP-14_W7.62mm_Socket_LongPads; Digikey (none) -> 296-1563-5-ND; LCSC C5586 -> (none); Mouser (none) -> 595-SN74HC00N
- U5: renamed from U4; footprint Package_SO:SOIC-16_3.9x9.9mm_P1.27mm -> Package_DIP:DIP-16_W7.62mm_Socket_LongPads; Digikey (none) -> 296-1575-5-ND; LCSC C5602 -> (none); Mouser (none) -> 595-SN74HC138N
- U7: Digikey (none) -> AT28C256-15PU-ND; Mouser (none) -> 556-AT28C25615PU
- U8: footprint Package_SO:SOIC-16_3.9x9.9mm_P1.27mm -> Package_DIP:DIP-16_W7.62mm_Socket_LongPads; Digikey (none) -> 296-1575-5-ND; LCSC C5602 -> (none)
- U9: footprint (none) -> Package_DIP:DIP-16_W7.62mm_Socket_LongPads; Digikey (none) -> 296-8246-5-ND; Mouser (none) -> 595-SN74HC163N
- X1: Digikey (none) -> X947-ND; Mouser (none) -> 815-ACO-16-EK; now in the parts list
- Y1: Digikey (none) -> 3155-1.8432M20P2/49U-ND; Mouser (none) -> 815-AB-1.8432-B2; now in the parts list
- renumbered J13 to J11
Connections:
- net A0: now also J16.18 (Pin_18)
- net A1: now also J16.16 (Pin_16)
- net A2: now also J16.14 (Pin_14)
- net D0: now also J16.17 (Pin_17)
- net D1: now also J16.15 (Pin_15)
- net D2: now also J16.13 (Pin_13)
- net D3: now also J16.11 (Pin_11)
- net D4: now also J16.9 (Pin_9)
- net D5: now also J16.7 (Pin_7)
- net D6: now also J16.5 (Pin_5)
- net D7: now also J16.3 (Pin_3)
- net GND: now also C10.2, C11.2, C12.2, C13.2, C14.2, C15.2, C16.2, C17.2, C18.2, C19.2, C20.2, C21.2, C22.2, C23.2, C24.2, C25.2, C26.2, C27.2, C28.2, C29.2, C30.2, C9.2, J10.2 (Pin_2), J16.1 (Pin_1), J16.20 (Pin_20), J20.2, J20.3, J21.2 (Pin_2), R36.2, TP1.1
- net RB: now also J16.8 (Pin_8)
- net RESB: now also J16.4 (Pin_4)
- net RWB: now also J16.6 (Pin_6)
- net VCC: now also C10.1, C11.1, C12.1, C13.1, C14.1, C15.1, C16.1, C17.1, C18.1, C19.1, C20.1, C21.1, C22.1, C23.1, C24.1, C25.1, C26.1, C27.1, C28.1, C29.1, C30.1, C9.1, D3.2 (A), J16.19 (Pin_19), J16.2 (Pin_2), J21.1 (Pin_1), J22.1 (Pin_1), R10.2, R12.2, R13.2, R14.2, R15.2, R4.2, R6.2, R8.2, SW11.1 (A), TP2.1
- net WB: now also J16.10 (Pin_10)
- net at C2.2, J12.1 (In), J13.1 (In): now also J10.1 (Pin_1)
- net IO1 renamed IO1B
- net IO1B: now also R4.1, SW1.16; no longer U5.15 (~{Y0})
- net IO2 renamed IO2B
- net IO2B: now also R6.1, SW1.15; no longer U5.14 (~{Y1})
- net IO3 renamed $8800
- net $8800: now also SW1.3; no longer U18.20 (~{CE})
- net IO4 renamed $8C00
- net $8C00: now also SW1.4
- net IO5 renamed $9000
- net $9000: now also SW1.5; no longer U21.3 (CS1B)
- net IO6 renamed $9400
- net $9400: now also SW1.6; no longer U11.23 (CS2B)
- net IO7 renamed $9800
- net $9800: now also SW1.7; no longer U19.8 (~{CS})
- net IO8 renamed $9C00
- net $9C00: now also SW1.8; no longer U8.2 (A1)
- new net: J20.1, SW11.2 (B)
- new net: D3.1 (K), J22.2 (Pin_2), R36.1
- new net $8000: SW1.1, U5.15 (~{Y0})
- new net $8400: SW1.2, U5.14 (~{Y1})
- new net IO3B: R8.1, SW1.14, U18.20 (~{CE})
- new net IO4B: J16.12 (Pin_12), R10.1, SW1.13
- new net IO5B: R12.1, SW1.12, U21.3 (CS1B)
- new net IO6B: R13.1, SW1.11, U11.23 (CS2B)
- new net IO7B: R14.1, SW1.10, U19.8 (~{CS})
- new net IO8B: R15.1, SW1.9, U8.2 (A1)
- no-connect marks 68 -> 32
Other:
- moved on the sheet: J14, J15, J3, J4, R2, R3, R5, R7, R9, U14E, U15B, U16E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

Commit message: Working on PCB
Parts:
- removed J6: PORT B, 6502-ACE:6502 GPIO Connector, symbol Connector_Generic:Conn_02x06_Odd_Even
- removed J8: PORT A, 6502-ACE:6502 GPIO Connector, symbol Connector_Generic:Conn_02x06_Odd_Even
- BT1: value BAT-HLD-001-THM -> CR2032
- J20: renamed from J16; footprint Connector_PinHeader_2.54mm:PinHeader_2x10_P2.54mm_Vertical -> Connector_PinHeader_2.54mm:PinHeader_2x10_P2.54mm_Horizontal
- X1: value OCXO-14 -> 16MHz
- renumbered C11 to C10, C13 to C11, C15 to C12, C17 to C13, C19 to C14, C21 to C15, C23 to C16, C25 to C17, C27 to C18, C29 to C19, C5 to C2, C10 to C20, C12 to C21, C14 to C22, C16 to C23, C18 to C24, C20 to C25, C22 to C26, C24 to C27, C26 to C28, C28 to C29, C6 to C3, C3 to C4, C7 to C5, C8 to C6, C4 to C7, C2 to C8, D3 to D1, D1 to D2, D2 to D3, J12 to J10, J17 to J11, J2 to J12, J10 to J14, J20 to J15, J14 to J16, J15 to J17, J21 to J18, J22 to J19, J18 to J2, J9 to J3, J19 to J4, J3 to J5, J11 to J6, J4 to J7, J5 to J8, J7 to J9, R2 to R1, R22 to R10, R24 to R11, R26 to R12, R28 to R13, R30 to R14, R11 to R15, R17 to R16, R19 to R17, R21 to R18, R23 to R19, R3 to R2, R25 to R20, R27 to R21, R29 to R22, R31 to R23, R34 to R24, R1 to R25, R36 to R26, R32 to R27, R35 to R28, R4 to R29, R5 to R3, R6 to R30, R8 to R31, R10 to R32, R12 to R33, R13 to R34, R14 to R35, R15 to R36, R7 to R4, R9 to R5, R33 to R6, R16 to R7, R18 to R8, R20 to R9, SW2 to SW1, SW13 to SW10, SW21 to SW11, SW30 to SW12, SW38 to SW13, SW47 to SW14, SW55 to SW15, SW63 to SW16, SW4 to SW17, SW14 to SW18, SW22 to SW19, SW12 to SW2, SW31 to SW20, SW39 to SW21, SW48 to SW22, SW56 to SW23, SW64 to SW24, SW5 to SW25, SW15 to SW26, SW23 to SW27, SW32 to SW28, SW40 to SW29, SW20 to SW3, SW49 to SW30, SW57 to SW31, SW65 to SW32, SW6 to SW33, SW16 to SW34, SW24 to SW35, SW33 to SW36, SW41 to SW37, SW50 to SW38, SW58 to SW39, SW29 to SW4, SW66 to SW40, SW42 to SW41, SW7 to SW42, SW17 to SW43, SW25 to SW44, SW34 to SW45, SW51 to SW46, SW59 to SW47, SW67 to SW48, SW43 to SW49, SW37 to SW5, SW8 to SW50, SW18 to SW51, SW26 to SW52, SW35 to SW53, SW44 to SW54, SW52 to SW55, SW60 to SW56, SW68 to SW57, SW9 to SW58, SW27 to SW59, SW46 to SW6, SW19 to SW60, SW36 to SW61, SW45 to SW62, SW53 to SW63, SW61 to SW64, SW69 to SW65, SW10 to SW66, SW28 to SW67, SW11 to SW68, SW1 to SW69, SW54 to SW7, SW62 to SW8, SW3 to SW9, TP2 to TP1, TP1 to TP2, U2 to U1, U22 to U10, U6 to U11, U14 to U12, U16 to U13, U4 to U14, U10 to U15, U1 to U16, U15 to U17, U5 to U19, U11 to U2, U8 to U20, U12 to U21, U13 to U22, U20 to U3, U21 to U4, U9 to U5, U17 to U6, U3 to U7, U7 to U8, U19 to U9
Other:
- moved on the sheet: J8, J9

Commit message: Change headers
Parts:
- J14, J18, J19, J3: footprint Connector_JST:JST_XH_B2B-XH-A_1x02_P2.50mm_Vertical -> Connector_PinHeader_2.54mm:PinHeader_1x02_P2.54mm_Vertical
Connections:
- net RDY: now also J20.6 (Pin_6)
- net RWB: no longer J20.6 (Pin_6)
Changed lines of the file:
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@@
 		)
 	)
-	(global_label "RWB"
-		(shape input)
+	(global_label "RDY"
+		(shape output)
 		(at 534.67 346.71 0)
 		(effects
@@
 			)
 		)
-		(property "Footprint" "Connector_JST:JST_XH_B2B-XH-A_1x02_P2.50mm_Vertical"
+		(property "Footprint" "Connector_PinHeader_2.54mm:PinHeader_1x02_P2.54mm_Vertical"
 			(at 637.54 260.35 0)
 			(hide yes)
@@
 			)
 		)
-		(property "Footprint" "Connector_JST:JST_XH_B2B-XH-A_1x02_P2.50mm_Vertical"
+		(property "Footprint" "Connector_PinHeader_2.54mm:PinHeader_1x02_P2.54mm_Vertical"
 			(at 374.65 88.9 0)
 			(hide yes)
@@
 			)
 		)
-		(property "Footprint" "Connector_JST:JST_XH_B2B-XH-A_1x02_P2.50mm_Vertical"
+		(property "Footprint" "Connector_PinHeader_2.54mm:PinHeader_1x02_P2.54mm_Vertical"
 			(at 637.54 274.32 0)
 			(hide yes)
@@
 			)
 		)
-		(property "Footprint" "Connector_JST:JST_XH_B2B-XH-A_1x02_P2.50mm_Vertical"
+		(property "Footprint" "Connector_PinHeader_2.54mm:PinHeader_1x02_P2.54mm_Vertical"
 			(at 412.75 201.93 0)
 			(hide yes)

Commit message: Finish PCB layout
Parts:
- added J5: VDD, Connector_PinHeader_2.54mm:PinHeader_1x02_P2.54mm_Vertical, symbol Connector_Generic:Conn_01x02
- J1: value PHI2 Select -> PHI2 SELECT
- J21: renamed from J20; footprint Connector_PinHeader_2.54mm:PinHeader_2x10_P2.54mm_Horizontal -> Connector_PinHeader_2.54mm:PinHeader_2x11_P2.54mm_Horizontal; symbol Connector_Generic:Conn_02x10_Odd_Even -> Connector_Generic:Conn_02x11_Odd_Even
- R10, R11, R12, R13, R14, R16, R17, R18, R19, R20, R21, R22, R23, R29, R30, R31, R32, R33, R34, R35, R36, R6, R7, R8, R9: value 1K -> 1k
- SW49: value R SHIFT -> SHIFT
- SW66: value R CTRL -> CTRL
- SW67: value R ALT -> ALT
- U3: footprint Package_DIP:DIP-40_W15.24mm_LongPads -> Package_DIP:DIP-40_W15.24mm_Socket_LongPads
- U6: footprint Package_DIP:DIP-40_W15.24mm -> Package_DIP:DIP-40_W15.24mm_Socket_LongPads
- renumbered J9 to J10, J10 to J11, J11 to J12, J12 to J13, J13 to J14, J14 to J15, J15 to J16, J16 to J17, J17 to J18, J18 to J19, J19 to J20, J5 to J6, J6 to J7, J7 to J8, J8 to J9
Connections:
- net A0: now also J21.20 (Pin_20); no longer J21.18 (Pin_18)
- net A1: now also J21.18 (Pin_18); no longer J21.16 (Pin_16)
- net A2: now also J21.16 (Pin_16); no longer J21.14 (Pin_14)
- net D0: now also J21.19 (Pin_19); no longer J21.17 (Pin_17)
- net D1: now also J21.17 (Pin_17); no longer J21.15 (Pin_15)
- net D2: now also J21.15 (Pin_15); no longer J21.13 (Pin_13)
- net D3: now also J21.13 (Pin_13); no longer J21.11 (Pin_11)
- net D4: now also J21.11 (Pin_11); no longer J21.9 (Pin_9)
- net D5: now also J21.9 (Pin_9); no longer J21.7 (Pin_7)
- net D6: now also J21.7 (Pin_7); no longer J21.5 (Pin_5)
- net D7: now also J21.5 (Pin_5); no longer J21.3 (Pin_3)
- net EXP2: now also U6.25 (PC3)
- net EXP3: now also U6.26 (PC4)
- net GND: now also J21.22 (Pin_22), J5.2 (Pin_2); no longer J21.20 (Pin_20)
- net HRDB: now also U6.27 (PC5)
- net IO4B: now also J21.14 (Pin_14); no longer J21.12 (Pin_12)
- net RB: now also J21.10 (Pin_10); no longer J21.8 (Pin_8)
- net RDY: now also J21.8 (Pin_8); no longer J21.6 (Pin_6)
- net RESB: now also J21.6 (Pin_6); no longer J21.4 (Pin_4)
- net VCC: now also J21.21 (Pin_21); no longer J21.19 (Pin_19)
- net WB: now also J21.12 (Pin_12); no longer J21.10 (Pin_10)
- net at U9.28 (VDD): now also J5.1 (Pin_1)
- net PREVB: now reaches U6.23 (PC1)
- net PREVB: now also J21.3 (Pin_3)
- net NEXTB: now reaches U6.24 (PC2)
- net NEXTB: now also J21.4 (Pin_4)
- no-connect marks 32 -> 26
Other:
- moved on the sheet: J3
