File: Hardware/ACE Board/Rev 1.0/ACE Board.kicad_pcb (KiCad board)
At the start: 2 copper layers, 335 x 250 mm, 203 parts, among them J1 PHI2 SELECT, J10 PORT A, J11 AUDIO L, J12 DB9 MALE (DTE), J13 PS/2, J14 AUDIO R, J15 AUDIO, J16 5V DC, J17 CART, J18 BUS, J19 VCC, J2 CTS EN, J20 POWER LED, J21 STORAGE, J3 RESET SW, J4 DCD EN, J5 VDD, J6 JOYSTICK A, J7 PADDLES, J8 JOYSTICK B, J9 PORT B, SW1 `, SW10 9, SW11 0, SW12 -, SW13 =, SW14 BACKSPACE, SW15 ESCAPE, SW16 TAB, SW17 Q, SW18 W, SW19 E, SW2 1, SW20 R, SW21 T, SW22 Y, SW23 U, SW24 I, SW25 O, SW26 P, SW27 [, SW28 ], SW29 \, SW3 2, SW30 INSERT, SW31 CAPS LOCK, SW32 A, SW33 S, SW34 D, SW35 F, SW36 G, SW37 H, SW38 J, SW39 K, SW4 3, SW40 L, SW41 SHIFT, SW42 ;, SW43 ', SW44 ENTER, SW45 DELETE, SW46 Z, SW47 X, SW48 C, SW49 SHIFT, SW5 4, SW50 V, SW51 B, SW52 N, SW53 M, SW54 ,, SW55 ., SW56 /, SW57 UP ARROW, SW58 CTRL, SW59 ALT, SW6 5, SW60 MENU, SW61 SPACE, SW62 FN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

Commit message: Working on PCB
Parts:
- moved Y1 29.3 mm to (157.5, 136.8), turned to -90 degrees
- moved C7 12.7 mm to (285.5, 123.6)
- moved C4 11.7 mm to (285.4, 117.3)
- moved J2 3.82 mm to (185.5, 129.2)
- moved C13 2.48 mm to (182.9, 157.1)
- moved R26 2.45 mm to (134.1, 114.8), turned to 0 degrees
- moved C12 0.89 mm to (149.8, 105.0)
- moved J1 0.10 mm to (218.5, 121.1)
Routing:
- net VCC: track 0.00 -> 1353.4 mm, vias 0 -> 48
- net PB5: track 412.0 -> 13.1 mm, vias 14 -> 2
- net PA7: track 404.8 -> 23.5 mm, vias 4 -> 2
- net PB2: track 386.9 -> 17.3 mm, vias 13 -> 2
- net PB0: track 373.9 -> 17.3 mm, vias 11 -> 2
- net PB4: track 351.5 -> 14.0 mm, vias 10 -> 2
- net PB6: track 350.5 -> 18.1 mm, vias 10 -> 2
- net PB7: track 331.4 -> 23.3 mm, vias 12 -> 2
- net PB1: track 315.6 -> 17.3 mm, vias 12 -> 2
- net PA1: track 311.9 -> 17.1 mm
- net PA5: track 277.1 -> 13.2 mm, vias 3 -> 2
- net PB3: track 266.2 -> 17.2 mm, vias 5 -> 2
- net PA6: track 246.7 -> 18.3 mm
- net PA3: track 192.9 -> 17.1 mm
- net PHI2: track 0.00 -> 169.9 mm, vias 0 -> 7
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