File: Hardware/ACE Board/Rev 1.0/ACE Board.kicad_pcb (KiCad board)
At the start: 2 copper layers, 335 x 250 mm, 203 parts, among them J1 PHI2 SELECT, J10 PORT A, J11 AUDIO L, J12 DB9 MALE (DTE), J13 PS/2, J14 AUDIO R, J15 AUDIO, J16 5V DC, J17 CART, J18 BUS, J19 VCC, J2 CTS EN, J20 POWER LED, J21 STORAGE, J3 RESET SW, J4 DCD EN, J5 VDD, J6 JOYSTICK A, J7 PADDLES, J8 JOYSTICK B, J9 PORT B, SW1 `, SW10 9, SW11 0, SW12 -, SW13 =, SW14 BACKSPACE, SW15 ESCAPE, SW16 TAB, SW17 Q, SW18 W, SW19 E, SW2 1, SW20 R, SW21 T, SW22 Y, SW23 U, SW24 I, SW25 O, SW26 P, SW27 [, SW28 ], SW29 \, SW3 2, SW30 INSERT, SW31 CAPS LOCK, SW32 A, SW33 S, SW34 D, SW35 F, SW36 G, SW37 H, SW38 J, SW39 K, SW4 3, SW40 L, SW41 SHIFT, SW42 ;, SW43 ', SW44 ENTER, SW45 DELETE, SW46 Z, SW47 X, SW48 C, SW49 SHIFT, SW5 4, SW50 V, SW51 B, SW52 N, SW53 M, SW54 ,, SW55 ., SW56 /, SW57 UP ARROW, SW58 CTRL, SW59 ALT, SW6 5, SW60 MENU, SW61 SPACE, SW62 FN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

Commit message: Finish ACE Board PCB
Parts:
- added J22: KEYBOARD, Connector_PinHeader_2.00mm:PinHeader_1x16_P2.00mm_Vertical, F.Cu at (281.5, 215.5)
- turned C23 to 90 degrees
- turned C25 to 0 degrees
- turned C26 to -90 degrees
Routing:
- net PB6: track 174.1 -> 849.0 mm, vias 7 -> 26
- net PB4: track 172.8 -> 826.5 mm, vias 6 -> 27
- net PB5: track 168.6 -> 800.8 mm, vias 7 -> 27
- net PB0: track 178.2 -> 787.5 mm, vias 6 -> 27
- net PB2: track 170.4 -> 777.1 mm, vias 8 -> 30
- net PB7: track 178.9 -> 778.5 mm, vias 8 -> 27
- net PB1: track 176.7 -> 733.2 mm, vias 8 -> 27
- net PB3: track 158.0 -> 691.8 mm, vias 5 -> 25
- net PA5: track 157.8 -> 682.9 mm, vias 8 -> 17
- net PA7: track 168.2 -> 690.5 mm, vias 6 -> 18
- net PA3: track 151.5 -> 639.4 mm, vias 6 -> 14
- net PA1: track 157.8 -> 623.4 mm, vias 8 -> 17
- net PA6: track 165.3 -> 567.4 mm, vias 8 -> 21
- net PA4: track 159.9 -> 488.1 mm, vias 8 -> 16
- net PA0: track 150.3 -> 450.7 mm, vias 9 -> 17
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