File: Hardware/ACE Board/Rev 1.0/ACE Board.kicad_pcb (KiCad board)
At the start: 2 copper layers, 335 x 250 mm, 203 parts, among them J1 PHI2 SELECT, J10 PORT A, J11 AUDIO L, J12 DB9 MALE (DTE), J13 PS/2, J14 KEYBOARD, J15 AUDIO R, J16 AUDIO, J17 5V DC, J18 CART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

Commit message: Ensure accurate Rev 1.0
Parts:
- R1, R2, R25, R3, R4: value 10k -> 1k
