File: Hardware/ACE Board/Rev 1.0/ACE Board.kicad_sch (KiCad schematic)
At the start: 186 parts, among them J1 PHI2 SELECT, J10 PORT A, J11 AUDIO L, J12 DB9 MALE (DTE), J13 PS/2, J14 AUDIO R, J15 AUDIO, J16 5V DC, J17 CART, J18 BUS, J19 VCC, J2 CTS EN, J20 POWER LED, J21 STORAGE, J3 RESET SW, J4 DCD EN, J5 VDD, J6 JOYSTICK A, J7 PADDLES, J8 JOYSTICK B, J9 PORT B, SW1 `, SW10 9, SW11 0, SW12 -, SW13 =, SW14 BACKSPACE, SW15 ESCAPE, SW16 TAB, SW17 Q, SW18 W, SW19 E, SW2 1, SW20 R, SW21 T, SW22 Y, SW23 U, SW24 I, SW25 O, SW26 P, SW27 [, SW28 ], SW29 \, SW3 2, SW30 INSERT, SW31 CAPS LOCK, SW32 A, SW33 S, SW34 D, SW35 F, SW36 G, SW37 H, SW38 J, SW39 K, SW4 3, SW40 L, SW41 SHIFT, SW42 ;, SW43 ', SW44 ENTER, SW45 DELETE, SW46 Z, SW47 X, SW48 C, SW49 SHIFT, SW5 4, SW50 V, SW51 B, SW52 N, SW53 M, SW54 ,, SW55 ., SW56 /, SW57 UP ARROW, SW58 CTRL, SW59 ALT, SW6 5, SW60 MENU, SW61 SPACE, SW62 FN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

Commit message: Update ACE project structure
Parts:
- BT1: footprint 6502-ACE:BAT_BAT-HLD-001-THM -> 6502 Parts:BAT_BAT-HLD-001-THM
- J10, J9: footprint 6502-ACE:6502 GPIO Connector -> 6502 Parts:6502 GPIO Connector
- J11, J14: footprint 6502-ACE:SWITCHCRAFT_PJRAN1X1U0XX -> 6502 Parts:SWITCHCRAFT_PJRAN1X1U0XX
- J13: footprint 6502-ACE:KMDGX-6S-BS -> 6502 Parts:KMDGX-6S-BS
- J17: footprint 6502-ACE:RHDR40W82P485X254_2X20_5740X93 -> 6502 Parts:RHDR40W82P485X254_2X20_5740X93
- J18: footprint 6502-ACE:6502 Bus Connector -> 6502 Parts:6502 Bus Connector
- SW1, SW10, SW11, SW12, SW13, SW15, SW17, SW18, SW19, SW2, SW20, SW21, SW22, SW23, SW24, SW25, SW26, SW27, SW28, SW3, SW30, SW32, SW33, SW34, SW35, SW36, SW37, SW38, SW39, SW4, SW40, SW42, SW43, SW45, SW46, SW47, SW48, SW5, SW50, SW51, SW52, SW53, SW54, SW55, SW56, SW57, SW6, SW60, SW63, SW64, SW65, SW7, SW8, SW9: footprint 6502-ACE:SW_Cherry_MX_1.00u_PCB -> 6502 Parts:SW_Cherry_MX_1.00u_PCB
- SW14: footprint 6502-ACE:SW_Cherry_MX_2.00u_PCB -> 6502 Parts:SW_Cherry_MX_2.00u_PCB
- SW16, SW29: footprint 6502-ACE:SW_Cherry_MX_1.50u_PCB -> 6502 Parts:SW_Cherry_MX_1.50u_PCB
- SW31: footprint 6502-ACE:SW_Cherry_MX_1.75u_PCB -> 6502 Parts:SW_Cherry_MX_1.75u_PCB
- SW41, SW44, SW49: footprint 6502-ACE:SW_Cherry_MX_2.25u_PCB -> 6502 Parts:SW_Cherry_MX_2.25u_PCB
- SW58, SW59, SW62, SW66, SW67: footprint 6502-ACE:SW_Cherry_MX_1.25u_PCB -> 6502 Parts:SW_Cherry_MX_1.25u_PCB
- SW61: footprint 6502-ACE:SW_Cherry_MX_6.25u_PCB -> 6502 Parts:SW_Cherry_MX_6.25u_PCB
- SW68: footprint 6502-ACE:SW_400MSP1R6BLKM6QE -> 6502 Parts:SW_400MSP1R6BLKM6QE
- U1: symbol 6502-ACE:65C02 -> 6502 Parts:65C02
- U15: symbol 6502-ACE:AS6C4008 -> 6502 Parts:AS6C4008
- U17: symbol 6502-ACE:74HC30 -> 6502 Parts:74HC30
- U18: symbol 6502-ACE:DS1511Y -> 6502 Parts:DS1511Y
- U2: symbol 6502-ACE:65C22 -> 6502 Parts:65C22
- U3: symbol 6502-ACE:Pico9918 -> 6502 Parts:Pico9918
- U4: symbol 6502-ACE:65C51 -> 6502 Parts:65C51
- U7: symbol 6502-ACE:AS6C62256 -> 6502 Parts:AS6C62256
- U8: symbol 6502-ACE:AT28C256 -> 6502 Parts:AT28C256
- U9: symbol 6502-ACE:6581 -> 6502 Parts:6581
Other:
- title: 6502 ACE -> 6502 ACE Board
- moved on the sheet: J5

Commit message: Updates to PCB
Parts:
- removed R15: 1k, Resistor_THT:R_Axial_DIN0204_L3.6mm_D1.6mm_P5.08mm_Horizontal, symbol Device:R
Connections:
- net VCC: now also U8.27 (~{WE})
Changed lines of the file:
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@@
 	)
 	(junction
+		(at 128.27 147.32)
+		(diameter 0)
+		(color 0 0 0 0)
+	)
+	(junction
 		(at 107.95 81.28)
 		(diameter 0)
@@
 	(wire
 		(pts
-			(xy 127 133.35) (xy 127 135.89)
-		)
-		(stroke
-			(width 0)
-			(type default)
-		)
-	)
-	(wire
-		(pts
 			(xy 492.76 55.88) (xy 497.84 55.88)
 		)
@@
 	(wire
 		(pts
+			(xy 128.27 147.32) (xy 137.16 147.32)
+		)
+		(stroke
+			(width 0)
+			(type default)
+		)
+	)
+	(wire
+		(pts
 			(xy 264.16 365.76) (xy 266.7 365.76)
 		)
@@
 	(wire
 		(pts
+			(xy 128.27 147.32) (xy 128.27 149.86)
+		)
+		(stroke
+			(width 0)
+			(type default)
+		)
+	)
+	(wire
+		(pts
 			(xy 746.76 129.54) (xy 749.3 129.54)
 		)
@@
 	(wire
 		(pts
-			(xy 127 149.86) (xy 125.73 149.86)
+			(xy 128.27 149.86) (xy 125.73 149.86)
 		)
 		(stroke
@@
 	(wire
 		(pts
-			(xy 127 143.51) (xy 127 149.86)
-		)
-		(stroke
-			(width 0)
-			(type default)
-		)
-	)
-	(wire
-		(pts
 			(xy 26.67 267.97) (xy 25.4 267.97)
 		)
@@
 	(wire
 		(pts
-			(xy 125.73 147.32) (xy 137.16 147.32)
+			(xy 125.73 147.32) (xy 128.27 147.32)
 		)
 		(stroke
@@
 		)
 	)
-	(global_label "VCC"
-		(shape input)
-		(at 127 133.35 90)
-		(effects
-			(font
-				(size 1.27 1.27)
-			)
-			(justify left)
-		)
-		(property "Intersheetrefs" "${INTERSHEET_REFS}"
-			(at 127 133.35 0)
-			(hide yes)
-			(show_name no)
-			(do_not_autoplace no)
-			(effects
-				(font
-					(size 1.27 1.27)
-				)
-			)
-		)
-	)
 	(global_label "D2"
 		(shape bidirectional)
@@
 					(unit 1)
 				)
-			)
-		)
-	)
-	(symbol
-		(lib_id "Device:R")
-		(at 127 139.7 180)
-		(unit 1)
-		(body_style 1)
-		(exclude_from_sim no)
-		(in_bom yes)
-		(on_board yes)
-		(in_pos_files yes)
-		(dnp no)
-		(property "Reference" "R15"
-			(at 124.714 140.97 0)
-			(show_name no)
-			(do_not_autoplace no)
-			(effects
-				(font
-					(size 1.27 1.27)
-				)
-				(justify left)
-			)
-		)
-		(property "Value" "1k"
-			(at 124.714 138.684 0)
-			(show_name no)
-			(do_not_autoplace no)
-			(effects
-				(font
-					(size 1.27 1.27)
-				)
-				(justify left)
-			)
-		)
-		(property "Footprint" "Resistor_THT:R_Axial_DIN0204_L3.6mm_D1.6mm_P5.08mm_Horizontal"
-			(at 128.778 139.7 90)
-			(hide yes)
-			(show_name no)
-			(do_not_autoplace no)
-			(effects
-				(font
-					(size 1.27 1.27)
-				)
-			)
-		)
-		(property "Datasheet" ""
-			(at 127 139.7 0)
-			(hide yes)
-			(show_name no)
-			(do_not_autoplace no)
-			(effects
-				(font
-					(size 1.27 1.27)
-				)
-			)
-		)
-		(property "Description" "Resistor"
-			(at 127 139.7 0)
-			(hide yes)
-			(show_name no)
-			(do_not_autoplace no)
-			(effects
-				(font
-					(size 1.27 1.27)
-				)
-			)
-		)
-		(pin "1"
-		)
-		(pin "2"
-		)
-		(instances
-			(project "ACE Board"
-				(path "/34a60d42-c14a-479d-bef3-5ff0ee57bad5"
-					(reference "R15")
-					(unit 1)
-				)

Commit message: Finish PCB layout
Parts:
- added SW70: RESET, Button_Switch_THT:SW_PUSH_6mm, symbol Switch:SW_Push
- U10: footprint Package_DIP:DIP-24_W7.62mm -> Package_DIP:DIP-24_W7.62mm_Socket_LongPads
Connections:
- net GND: now also SW70.2
- net at J3.1 (Pin_1), U6.22 (PC0): now also SW70.1
Changed lines of the file:
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@@
 	)
 	(junction
+		(at 369.57 88.9)
+		(diameter 0)
+		(color 0 0 0 0)
+	)
+	(junction
 		(at 673.1 133.35)
 		(diameter 0)
@@
 	(wire
 		(pts
+			(xy 387.35 68.58) (xy 387.35 72.39)
+		)
+		(stroke
+			(width 0)
+			(type default)
+		)
+	)
+	(wire
+		(pts
 			(xy 496.57 251.46) (xy 500.38 251.46)
 		)
@@
 	(wire
 		(pts
-			(xy 355.6 88.9) (xy 374.65 88.9)
+			(xy 355.6 88.9) (xy 369.57 88.9)
 		)
 		(stroke
@@
 	(wire
 		(pts
+			(xy 369.57 68.58) (xy 369.57 88.9)
+		)
+		(stroke
+			(width 0)
+			(type default)
+		)
+	)
+	(wire
+		(pts
 			(xy 665.48 177.8) (xy 668.02 177.8)
 		)
@@
 	(wire
 		(pts
+			(xy 374.65 68.58) (xy 369.57 68.58)
+		)
+		(stroke
+			(width 0)
+			(type default)
+		)
+	)
+	(wire
+		(pts
 			(xy 769.62 129.54) (xy 769.62 146.05)
 		)
@@
 	(wire
 		(pts
+			(xy 369.57 88.9) (xy 374.65 88.9)
+		)
+		(stroke
+			(width 0)
+			(type default)
+		)
+	)
+	(wire
+		(pts
 			(xy 452.12 199.39) (xy 452.12 184.15)
 		)
@@
 	(wire
 		(pts
+			(xy 384.81 68.58) (xy 387.35 68.58)
+		)
+		(stroke
+			(width 0)
+			(type default)
+		)
+	)
+	(wire
+		(pts
 			(xy 58.42 250.19) (xy 60.96 250.19)
 		)
@@
 	)
 	(symbol
+		(lib_id "power:GND")
+		(at 387.35 72.39 0)
+		(unit 1)
+		(body_style 1)
+		(exclude_from_sim no)
+		(in_bom yes)
+		(on_board yes)
+		(in_pos_files yes)
+		(dnp no)
+		(fields_autoplaced yes)
+		(property "Reference" "#PWR042"
+			(at 387.35 78.74 0)
+			(hide yes)
+			(show_name no)
+			(do_not_autoplace no)
+			(effects
+				(font
+					(size 1.27 1.27)
+				)
+			)
+		)
+		(property "Value" "GND"
+			(at 387.35 77.47 0)
+			(show_name no)
+			(do_not_autoplace no)
+			(effects
+				(font
+					(size 1.27 1.27)
+				)
+			)
+		)
+		(property "Footprint" ""
+			(at 387.35 72.39 0)
+			(hide yes)
+			(show_name no)
+			(do_not_autoplace no)
+			(effects
+				(font
+					(size 1.27 1.27)
+				)
+			)
+		)
+		(property "Datasheet" ""
+			(at 387.35 72.39 0)
+			(hide yes)
+			(show_name no)
+			(do_not_autoplace no)
+			(effects
+				(font
+					(size 1.27 1.27)
+				)
+			)
+		)
+		(property "Description" "Power symbol creates a global label with name \"GND\" , ground"
+			(at 387.35 72.39 0)
+			(hide yes)
+			(show_name no)
+			(do_not_autoplace no)
+			(effects
+				(font
+					(size 1.27 1.27)
+				)
+			)
+		)
+		(pin "1"
+		)
+		(instances
+			(project "ACE Board"
+				(path "/34a60d42-c14a-479d-bef3-5ff0ee57bad5"
+					(reference "#PWR042")
+					(unit 1)
+				)
+			)
+		)
+	)
+	(symbol
 		(lib_id "Oscillator:OCXO-14")
 		(at 93.98 86.36 0)
@@
 	)
 	(symbol
+		(lib_id "Switch:SW_Push")
+		(at 379.73 68.58 0)
+		(unit 1)
+		(body_style 1)
+		(exclude_from_sim no)
+		(in_bom yes)
+		(on_board yes)
+		(in_pos_files yes)
+		(dnp no)
+		(fields_autoplaced yes)
+		(property "Reference" "SW70"
+			(at 379.73 60.96 0)
+			(show_name no)
+			(do_not_autoplace no)
+			(effects
+				(font
+					(size 1.27 1.27)
+				)
+			)
+		)
+		(property "Value" "RESET"
+			(at 379.73 63.5 0)
+			(show_name no)
+			(do_not_autoplace no)
+			(effects
+				(font
+					(size 1.27 1.27)
+				)
+			)
+		)
+		(property "Footprint" "Button_Switch_THT:SW_PUSH_6mm"
+			(at 379.73 63.5 0)
+			(hide yes)
+			(show_name no)
+			(do_not_autoplace no)
+			(effects
+				(font
+					(size 1.27 1.27)
+				)
+			)
+		)
+		(property "Datasheet" ""
+			(at 379.73 63.5 0)
+			(hide yes)
+			(show_name no)
+			(do_not_autoplace no)
+			(effects
+				(font
+					(size 1.27 1.27)
+				)
+			)
+		)
+		(property "Description" "Push button switch, generic, two pins"
+			(at 379.73 68.58 0)
+			(hide yes)
+			(show_name no)
+			(do_not_autoplace no)
+			(effects
+				(font
+					(size 1.27 1.27)
+				)
+			)
+		)
+		(pin "2"
+		)
+		(pin "1"
+		)
+		(instances
+			(project "ACE Board"
+				(path "/34a60d42-c14a-479d-bef3-5ff0ee57bad5"
+					(reference "SW70")
+					(unit 1)
+				)
+			)
+		)
+	)
+	(symbol
 		(lib_id "power:GND")
 		(at 95.25 193.04 0)
@@
 			)
 		)
-		(property "Footprint" "Package_DIP:DIP-24_W7.62mm"
+		(property "Footprint" "Package_DIP:DIP-24_W7.62mm_Socket_LongPads"
 			(at 513.08 204.47 0)
 			(hide yes)

Commit message: Change storage header
Parts:
- J21: footprint Connector_PinHeader_2.54mm:PinHeader_2x11_P2.54mm_Horizontal -> Connector_PinSocket_2.54mm:PinSocket_2x10_P2.54mm_Horizontal; symbol Connector_Generic:Conn_02x11_Odd_Even -> Connector_Generic:Conn_02x10_Odd_Even; Digikey (none) -> S5563-ND; MPN (none) -> PPPC102LJBN-RC
Connections:
- net A0: now also J21.18 (Pin_18); no longer J21.20 (Pin_20)
- net A1: now also J21.16 (Pin_16); no longer J21.18 (Pin_18)
- net A2: now also J21.14 (Pin_14); no longer J21.16 (Pin_16)
- net D0: now also J21.17 (Pin_17); no longer J21.19 (Pin_19)
- net D1: now also J21.15 (Pin_15); no longer J21.17 (Pin_17)
- net D2: now also J21.13 (Pin_13); no longer J21.15 (Pin_15)
- net D3: now also J21.11 (Pin_11); no longer J21.13 (Pin_13)
- net D4: now also J21.9 (Pin_9); no longer J21.11 (Pin_11)
- net D5: now also J21.7 (Pin_7); no longer J21.9 (Pin_9)
- net D6: now also J21.5 (Pin_5); no longer J21.7 (Pin_7)
- net D7: now also J21.3 (Pin_3); no longer J21.5 (Pin_5)
- net EXP2: no longer U6.25 (PC3)
- net EXP3: no longer U6.26 (PC4)
- net GND: now also J21.20 (Pin_20); no longer J21.22 (Pin_22)
- net HRDB: no longer U6.27 (PC5)
- net IO4B: now also J21.12 (Pin_12); no longer J21.14 (Pin_14)
- net IRQB: no longer U6.28 (PC6)
- net NMIB: now also U6.21 (PD7); no longer U6.29 (PC7)
- net RB: now also J21.8 (Pin_8); no longer J21.10 (Pin_10)
- net RDY: now also J21.6 (Pin_6); no longer J21.8 (Pin_8)
- net RESB: now also J21.4 (Pin_4), U6.29 (PC7); no longer J21.6 (Pin_6), U6.21 (PD7)
- net VCC: now also J21.19 (Pin_19); no longer J21.21 (Pin_21)
- net WB: now also J21.10 (Pin_10); no longer J21.12 (Pin_12)
- net NEXTB: no longer names the net of U6.24 (PC2)
- net NEXTB: no longer J21.4 (Pin_4)
- net PREVB: no longer names the net of U6.23 (PC1)
- net PREVB: no longer J21.3 (Pin_3)
- no-connect marks 26 -> 32
Other:
- moved on the sheet: J3, SW70

Commit message: Finish ACE Board PCB
Parts:
- added J22: KEYBOARD, Connector_PinHeader_2.00mm:PinHeader_1x16_P2.00mm_Vertical, symbol Connector_Generic:Conn_01x16
Connections:
- net PA0: now also J22.1 (Pin_1)
- net PA1: now also J22.2 (Pin_2)
- net PA2: now also J22.3 (Pin_3)
- net PA3: now also J22.4 (Pin_4)
- net PA4: now also J22.5 (Pin_5)
- net PA5: now also J22.6 (Pin_6)
- net PA6: now also J22.7 (Pin_7)
- net PA7: now also J22.8 (Pin_8)
- net PB0: now also J22.9 (Pin_9)
- net PB1: now also J22.10 (Pin_10)
- net PB2: now also J22.11 (Pin_11)
- net PB3: now also J22.12 (Pin_12)
- net PB4: now also J22.13 (Pin_13)
- net PB5: now also J22.14 (Pin_14)
- net PB6: now also J22.15 (Pin_15)
- net PB7: now also J22.16 (Pin_16)

Commit message: Add BOMs
Parts:
- D2, D3: Amazon https://www.amazon.com/gp/product/B0CKSNPVH8 -> (none); Other (none) -> https://www.amazon.com/gp/product/B0CKSNPVH8
- J13: Amazon https://www.amazon.com/dp/B08GS3QL7T -> (none); Other (none) -> https://www.amazon.com/dp/B08GS3QL7T
- SW69: Amazon https://www.amazon.com/Yohii-2-54mm-Positions-Double-Assort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 -> (none); Other (none) -> https://www.amazon.com/Yohii-2-54mm-Positions-Double-Assort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
- TP1, TP2: now left out of the parts list

Commit message: Finish BOM and add to README
Parts:
- C1, C10, C11, C12, C13, C14, C15, C16, C17, C18, C19, C20, C21, C22, C23, C24, C25, C26, C27, C28, C29, C30, C9: Digikey (none) -> 478-5732-ND
- C2, C3, C5, C6, C8: Digikey (none) -> 478-7667-ND
- C4, C7: Digikey (none) -> 478-SR151C222KAATR1CT-ND
- D1: Digikey (none) -> 732-5008-ND; Other (none) -> https://www.amazon.com/300-Pcs-LED-Diode-Assortment/dp/B0F3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
- J1, J15, J19, J2, J20, J22, J3, J4, J5, J7: Other (none) -> https://www.amazon.com/Straight-Breakaway-Connector-Breadbo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
- J10, J9: Digikey (none) -> 2057-BHR-12-VUA-ND; Other (none) -> https://www.amazon.com/uxcell-2-54mm-2x6-Pin-Straight-Conne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
- R1, R10, R11, R12, R13, R14, R16, R17, R18, R19, R2, R20, R21, R22, R23, R24, R25, R27, R28, R29, R3, R30, R31, R32, R33, R34, R35, R36, R4, R5, R6, R7, R8, R9: Digikey (none) -> RNF18FTD1K00CT-ND; Other (none) -> https://www.amazon.com/ALLECIN-8W-Metal-Film-Resistor/dp/B0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
- R26: Other (none) -> https://www.amazon.com/ALLECIN-8W-Metal-Film-Resistor/dp/B0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
- SW1, SW10, SW11, SW12, SW13, SW14, SW15, SW16, SW17, SW18, SW19, SW2, SW20, SW21, SW22, SW23, SW24, SW25, SW26, SW27, SW28, SW29, SW3, SW30, SW31, SW32, SW33, SW34, SW35, SW36, SW37, SW38, SW39, SW4, SW40, SW41, SW42, SW43, SW44, SW45, SW46, SW47, SW48, SW49, SW5, SW51, SW52, SW53, SW54, SW55, SW56, SW57, SW58, SW59, SW6, SW60, SW61, SW62, SW63, SW64, SW65, SW66, SW67, SW7, SW8, SW9: Digikey (none) -> CH196-ND; Other (none) -> https://www.amazon.com/dp/B0FYR5TV3X
- SW50: Digikey (none) -> CH196-ND; Other (none) -> https://www.amazon.com/dp/B0FYR5TV3Xhttps://www.amazon.com/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
- SW70: Other (none) -> https://www.amazon.com/QTEATAK-Momentary-Tactile-Button-Swi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
- U3: Other (none) -> https://www.tindie.com/products/visrealm/pico9918-pro/
- U4: Other (none) -> https://www.jameco.com/z/R6551AP-Rockwell-IC-6551-Asynchron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
- U9: Other (none) -> https://retrocomp.cz/produkt?id=2

Commit message: Update BOM
Parts:
- C1, C10, C11, C12, C13, C14, C15, C16, C17, C18, C19, C2, C20, C21, C22, C23, C24, C25, C26, C27, C28, C29, C3, C30, C4, C5, C6, C7, C8, C9: Other (none) -> https://www.amazon.com/PANMILED-Multilayer-Monolithic-Capac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
- J18: Other (none) -> https://www.amazon.com/Female-Headers-Connector-Header-Rasp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
