File: Hardware/ACE CF Adapter/Rev 1.0/ACE CF Adapter.kicad_pcb (KiCad board)
At the start: 2 copper layers, 75 x 50 mm, 15 parts, among them J21 STORAGE, J3 Compact Flash

Commit message: Change storage header
Parts:
- J21: footprint Connector_PinSocket_2.54mm:PinSocket_2x11_P2.54mm_Horizontal -> Connector_PinHeader_2.54mm:PinHeader_2x10_P2.54mm_Horizontal
- moved J21 24.9 mm to (148.9, 113.3), turned to -90 degrees
- moved R3 18.1 mm to (134.7, 106.0), turned to 180 degrees
- moved R4 8.04 mm to (122.0, 102.5), turned to 0 degrees
- moved R2 2.25 mm to (139.8, 102.5)
- moved J3 0.13 mm to (137.5, 84.0)
- moved R1 0.09 mm to (144.8, 102.5)
Connections:
- J21 pad 10: RB -> WB
- J21 pad 11: D4 -> D3
- J21 pad 12: WB -> IO4B
- J21 pad 13: D3 -> D2
- J21 pad 14: IO4B -> A2
- J21 pad 15: D2 -> D1
- J21 pad 16: A2 -> A1
- J21 pad 17: D1 -> D0
- J21 pad 18: A1 -> A0
- J21 pad 19: D0 -> VCC
- J21 pad 20: A0 -> GND
- J21 pad 3: unconnected-(J21-Pin_3-Pad3) -> D7
- J21 pad 4: unconnected-(J21-Pin_4-Pad4) -> RESB
- J21 pad 5: D7 -> D6
- J21 pad 6: RESB -> unconnected-(J21-Pin_6-Pad6)
- J21 pad 7: D6 -> D5
- J21 pad 8: unconnected-(J21-Pin_8-Pad8) -> RB
- J21 pad 9: D5 -> D4
Routing:
- net WB: track 53.2 -> 22.9 mm, vias 4 -> 2
- net RB: track 50.7 -> 21.7 mm, vias 4 -> 2
- net IO4B: track 49.9 -> 29.6 mm, vias 4 -> 2
- net D7: track 36.8 -> 16.6 mm, vias 4 -> 0
- net VCC: track 64.4 -> 78.0 mm, vias 4 -> 6
- net A0: track 32.5 -> 21.0 mm
- net D4: track 38.0 -> 29.0 mm, vias 4 -> 2
- net D1: track 28.4 -> 21.5 mm
- net D0: track 30.3 -> 23.8 mm, vias 2 -> 4
- net RESB: track 37.3 -> 31.2 mm, vias 4 -> 2
- net D3: track 36.0 -> 31.6 mm
- net A1: track 25.6 -> 21.2 mm
- net D6: track 26.1 -> 21.9 mm, vias 4 -> 2
- net Net-(J3-~{REG}): track 13.4 -> 9.18 mm, vias 2 -> 0
- net D5: track 27.3 -> 24.1 mm, vias 4 -> 2
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
Commit message: Add BOMs
Parts:
- renumbered J21 to J1, J3 to J2
Changed lines of the file:
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@@
 		(descr "101D-TAAB-R01-8")
 		(tags "Connector")
-		(property "Reference" "J3"
+		(property "Reference" "J2"
 			(at 0 0.55 0)
 			(layer "F.SilkS")
@@
 			)
 		)
-		(attr through_hole)
+		(attr through_hole exclude_from_bom)
 		(duplicate_pad_numbers_are_jumpers no)
 		(fp_line
@@
 			(size 0.4 2.5)
 			(layers "F.Cu" "F.Mask" "F.Paste")
-			(net "unconnected-(J3-~{IOCS16}-Pad24)")
+			(net "unconnected-(J2-~{IOCS16}-Pad24)")
 			(pinfunction "~{IOCS16}_24")
 			(pintype "output+no_connect")
@@
 			(size 0.4 2.5)
 			(layers "F.Cu" "F.Mask" "F.Paste")
-			(net "unconnected-(J3-~{CD2}-Pad25)")
+			(net "unconnected-(J2-~{CD2}-Pad25)")
 			(pinfunction "~{CD2}_25")
 			(pintype "output+no_connect")
@@
 			(size 0.4 2.5)
 			(layers "F.Cu" "F.Mask" "F.Paste")
-			(net "unconnected-(J3-~{CD1}-Pad26)")
+			(net "unconnected-(J2-~{CD1}-Pad26)")
 			(pinfunction "~{CD1}_26")
 			(pintype "output+no_connect")
@@
 			(size 0.4 2.5)
 			(layers "F.Cu" "F.Mask" "F.Paste")
-			(net "unconnected-(J3-D11-Pad27)")
+			(net "unconnected-(J2-D11-Pad27)")
 			(pinfunction "D11_27")
 			(pintype "bidirectional+no_connect")
@@
 			(size 0.4 2.5)
 			(layers "F.Cu" "F.Mask" "F.Paste")
-			(net "unconnected-(J3-D12-Pad28)")
+			(net "unconnected-(J2-D12-Pad28)")
 			(pinfunction "D12_28")
 			(pintype "bidirectional+no_connect")
@@
 			(size 0.4 2.5)
 			(layers "F.Cu" "F.Mask" "F.Paste")
-			(net "unconnected-(J3-D13-Pad29)")
+			(net "unconnected-(J2-D13-Pad29)")
 			(pinfunction "D13_29")
 			(pintype "bidirectional+no_connect")
@@
 			(size 0.4 2.5)
 			(layers "F.Cu" "F.Mask" "F.Paste")
-			(net "unconnected-(J3-D14-Pad30)")
+			(net "unconnected-(J2-D14-Pad30)")
 			(pinfunction "D14_30")
 			(pintype "bidirectional+no_connect")
@@
 			(size 0.4 2.5)
 			(layers "F.Cu" "F.Mask" "F.Paste")
-			(net "unconnected-(J3-D15-Pad31)")
+			(net "unconnected-(J2-D15-Pad31)")
 			(pinfunction "D15_31")
 			(pintype "bidirectional+no_connect")
@@
 			(size 0.4 2.5)
 			(layers "F.Cu" "F.Mask" "F.Paste")
-			(net "Net-(J3-~{CS1})")
+			(net "Net-(J2-~{CS1})")
 			(pinfunction "~{CS1}_32")
 			(pintype "input")
@@
 			(size 0.4 2.5)
 			(layers "F.Cu" "F.Mask" "F.Paste")
-			(net "unconnected-(J3-~{VS1}-Pad33)")
+			(net "unconnected-(J2-~{VS1}-Pad33)")
 			(pinfunction "~{VS1}_33")
 			(pintype "output+no_connect")
@@
 			(size 0.4 2.5)
 			(layers "F.Cu" "F.Mask" "F.Paste")
-			(net "Net-(J3-~{WE})")
+			(net "Net-(J2-~{WE})")
 			(pinfunction "~{WE}_36")
 			(pintype "input")
@@
 			(size 0.4 2.5)
 			(layers "F.Cu" "F.Mask" "F.Paste")
-			(net "unconnected-(J3-INTRQ-Pad37)")
+			(net "unconnected-(J2-INTRQ-Pad37)")
 			(pinfunction "INTRQ_37")
 			(pintype "output+no_connect")
@@
 			(size 0.4 2.5)
 			(layers "F.Cu" "F.Mask" "F.Paste")
-			(net "unconnected-(J3-~{VS2}-Pad40)")
+			(net "unconnected-(J2-~{VS2}-Pad40)")
 			(pinfunction "~{VS2}_40")
 			(pintype "input+no_connect")
@@
 			(size 0.4 2.5)
 			(layers "F.Cu" "F.Mask" "F.Paste")
-			(net "unconnected-(J3-IORDY-Pad42)")
+			(net "unconnected-(J2-IORDY-Pad42)")
 			(pinfunction "IORDY_42")
 			(pintype "output+no_connect")
@@
 			(size 0.4 2.5)
 			(layers "F.Cu" "F.Mask" "F.Paste")
-			(net "unconnected-(J3-NC-Pad43)")
+			(net "unconnected-(J2-NC-Pad43)")
 			(pinfunction "NC_43")
 			(pintype "no_connect")
@@
 			(size 0.4 2.5)
 			(layers "F.Cu" "F.Mask" "F.Paste")
-			(net "Net-(J3-~{REG})")
+			(net "Net-(J2-~{REG})")
 			(pinfunction "~{REG}_44")
 			(pintype "input")
@@
 			(size 0.4 2.5)
 			(layers "F.Cu" "F.Mask" "F.Paste")
-			(net "Net-(J3-~{DASP})")
+			(net "Net-(J2-~{DASP})")
 			(pinfunction "~{DASP}_45")
 			(pintype "bidirectional")
@@
 			(size 0.4 2.5)
 			(layers "F.Cu" "F.Mask" "F.Paste")
-			(net "Net-(J3-~{PDIAG})")
+			(net "Net-(J2-~{PDIAG})")
 			(pinfunction "~{PDIAG}_46")
 			(pintype "bidirectional")
@@
 			(size 0.4 2.5)
 			(layers "F.Cu" "F.Mask" "F.Paste")
-			(net "unconnected-(J3-D8-Pad47)")
+			(net "unconnected-(J2-D8-Pad47)")
 			(pinfunction "D8_47")
 			(pintype "bidirectional+no_connect")
@@
 			(size 0.4 2.5)
 			(layers "F.Cu" "F.Mask" "F.Paste")
-			(net "unconnected-(J3-D9-Pad48)")
+			(net "unconnected-(J2-D9-Pad48)")
 			(pinfunction "D9_48")
 			(pintype "bidirectional+no_connect")
@@
 			(size 0.4 2.5)
 			(layers "F.Cu" "F.Mask" "F.Paste")
-			(net "unconnected-(J3-D10-Pad49)")
+			(net "unconnected-(J2-D10-Pad49)")
 			(pinfunction "D10_49")
 			(pintype "bidirectional+no_connect")
@@
 			(layers "*.Cu" "*.Mask")
 			(remove_unused_layers no)
-			(net "Net-(J3-~{REG})")
+			(net "Net-(J2-~{REG})")
 			(pintype "passive")
 		)
@@
 			(layers "*.Cu" "*.Mask")
 			(remove_unused_layers no)
-			(net "Net-(J3-~{CS1})")
+			(net "Net-(J2-~{CS1})")
 			(pintype "passive")
 		)
@@
 			(layers "*.Cu" "*.Mask")
 			(remove_unused_layers no)
-			(net "Net-(J3-~{WE})")
+			(net "Net-(J2-~{WE})")
 			(pintype "passive")
 		)
@@
 			(layers "*.Cu" "*.Mask")
 			(remove_unused_layers no)
-			(net "Net-(J3-~{PDIAG})")
+			(net "Net-(J2-~{PDIAG})")
 			(pintype "passive")
 		)
@@
 		(descr "Through hole angled pin header, 2x10, 2.54mm pitch, 6mm pin length, double rows")
 		(tags "Through hole angled pin header THT 2x10 2.54mm double row")
-		(property "Reference" "J21"
+		(property "Reference" "J1"
 			(at 5.16 -2.57 90)
 			(layer "F.SilkS")
@@
 			(layers "*.Cu" "*.Mask")
 			(remove_unused_layers no)
-			(net "unconnected-(J21-Pin_6-Pad6)")
+			(net "unconnected-(J1-Pin_6-Pad6)")
 			(pinfunction "Pin_6_6")
 			(pintype "passive+no_connect")
@@
 			(layers "*.Cu" "*.Mask")
 			(remove_unused_layers no)
-			(net "Net-(J3-~{DASP})")
+			(net "Net-(J2-~{DASP})")
 			(pintype "passive")
 		)
@@
 	)
 	(segment
-		(start 144.803 96.85)
-		(end 144.803 102.383)
-		(width 0.2)
-		(layer "F.Cu")
-		(net "Net-(J3-~{CS1})")
-	)
-	(segment
 		(start 142.263 96.85)
 		(end 142.263 109.147)
@@
 	)
 	(segment
-		(start 139.75 102.5)
-		(end 139.75 96.877)
-		(width 0.2)
-		(layer "F.Cu")
-		(net "Net-(J3-~{WE})")
-	)
-	(segment
-		(start 139.75 96.877)
-		(end 139.723 96.85)
-		(width 0.2)
-		(layer "F.Cu")
-		(net "Net-(J3-~{WE})")
-	)
-	(segment
 		(start 145.11 114.55)
 		(end 146.38 115.82)
@@
 	)
 	(segment
-		(start 129.59 96.878)
-		(end 129.562 96.85)
-		(width 0.2)
-		(layer "F.Cu")
-		(net "Net-(J3-~{REG})")
-	)
-	(segment
-		(start 129.59 106.02)
-		(end 129.59 96.878)
+		(start 144.803 96.85)
+		(end 144.803 102.383)
 		(width 0.2)
 		(layer "F.Cu")
-		(net "Net-(J3-~{REG})")
+		(net "Net-(J2-~{CS1})")
 	)
 	(segment
@@
 		(width 0.2)
 		(layer "F.Cu")
-		(net "Net-(J3-~{DASP})")
+		(net "Net-(J2-~{DASP})")
 	)
 	(segment
@@
 		(width 0.2)
 		(layer "F.Cu")
-		(net "Net-(J3-~{DASP})")
+		(net "Net-(J2-~{DASP})")
 	)
 	(segment
@@
 		(width 0.2)
 		(layer "F.Cu")
-		(net "Net-(J3-~{DASP})")
+		(net "Net-(J2-~{DASP})")
 	)
 	(segment
@@
 		(width 0.2)
 		(layer "F.Cu")
-		(net "Net-(J3-~{DASP})")
+		(net "Net-(J2-~{DASP})")
 	)
 	(segment
@@
 		(width 0.2)
 		(layer "F.Cu")
-		(net "Net-(J3-~{DASP})")
+		(net "Net-(J2-~{DASP})")
 	)
 	(via
@@
 		(drill 0.3)
 		(layers "F.Cu" "B.Cu")
-		(net "Net-(J3-~{DASP})")
+		(net "Net-(J2-~{DASP})")
 	)
 	(via
@@
 		(drill 0.3)
 		(layers "F.Cu" "B.Cu")
-		(net "Net-(J3-~{DASP})")
+		(net "Net-(J2-~{DASP})")
 	)
 	(segment
@@
 		(width 0.2)
 		(layer "B.Cu")
-		(net "Net-(J3-~{DASP})")
+		(net "Net-(J2-~{DASP})")
+	)
+	(segment
+		(start 139.75 102.5)
+		(end 139.75 96.877)
+		(width 0.2)
+		(layer "F.Cu")
+		(net "Net-(J2-~{WE})")
+	)
+	(segment
+		(start 139.75 96.877)
+		(end 139.723 96.85)
+		(width 0.2)
+		(layer "F.Cu")
+		(net "Net-(J2-~{WE})")
+	)
+	(segment
+		(start 129.59 96.878)
+		(end 129.562 96.85)
+		(width 0.2)
+		(layer "F.Cu")
+		(net "Net-(J2-~{REG})")
+	)
+	(segment
+		(start 129.59 106.02)
+		(end 129.59 96.878)
+		(width 0.2)
+		(layer "F.Cu")
+		(net "Net-(J2-~{REG})")
 	)
 	(segment
@@
 		(width 0.2)
 		(layer "F.Cu")
-		(net "Net-(J3-~{PDIAG})")
+		(net "Net-(J2-~{PDIAG})")
 	)
 	(segment
@@
 		(width 0.2)
 		(layer "F.Cu")
-		(net "Net-(J3-~{PDIAG})")
+		(net "Net-(J2-~{PDIAG})")
 	)
 	(zone
