File: Hardware/ACE RAM Patch/Rev 1.1/ACE RAM Patch.kicad_sch (KiCad schematic)
At the start: 4 parts, among them J1 74HC00 (U12), J2 74HC00 (U13), U1 74HC00, U2 74HC02

Commit message: ACE RAM Patch Rev 1.1: lay it out to mount under the ACE
U12 and U13 come off the Rev 1.0 board, chips and sockets, and the patch is
soldered underneath on pin headers, front side up. U1, J1, J2 and U2 sit in
one row, 92.6 x 13.1 mm: J1 and J2 on the front, into U12's and U13's holes,
and U1 and U2 on the back, hanging below. J2 is 23.00 mm from J1, and all 28
header pins land on U12's and U13's pads on the Rev 1.0 board to 0.0000 mm.

No DRC errors, nothing unconnected, no schematic parity issues, and power
flags clear the schematic's ERC. Production files are generated as Rev 1.1,
and their gerbers and drill files match the board shape for shape.

Co-Authored-By: Claude Opus 5.5 (1M context) <noreply@anthropic.com>
Other:
- note added: "Fitting: take U12 and U13, chips and sockets, off the Rev 1.0 ACE Board. The patch mounts underneath it, front side up: pin headers from J1 go into U12's holes and from J2 into U13's, soldered on both boards. U1 and U2 are on the back, hanging below; trim their leads flush on the front. U13's pin 1 is 23.00 mm from U12's along the row, so J2 sits 23.00 mm from J1. LOADL and LOADH go high only on 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"
- note removed: "Fitting: take the 74HC00s out of U12 and U13 on the Rev 1.0 ACE Board. J1 plugs into U12's socket and J2 into U13's. Both sockets face the same way, and U13's pin 1 is 23.00 mm from U12's pin 1 along the row, so J2 sits 23.00 mm from J1 on the patch. LOADL and LOADH go high only on a write to the bank register, $83FF or $87FF, while PHI2 is high: A9·A8·(A0-A7 all ones), with IO1 for LOADL and B18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"
