File: Hardware/ACE Board/Rev 1.1/ACE Board.kicad_pcb (KiCad board)
At the start: 2 copper layers, 335 x 250 mm, 205 parts, among them J1 CTS EN, J10 AUDIO L, J11 DB9 MALE (DTE), J12 PS/2, J13 KEYBOARD, J14 AUDIO R, J15 AUDIO, J16 5V DC, J17 CART, J18 BUS, J19 VCC, J2 RESET SW, J20 POWER LED, J21 STORAGE, J3 DCD EN, J4 VDD, J5 JOYSTICK A, J6 PADDLES, J7 JOYSTICK B, J8 PORT B, J9 PORT A, SW1 `, SW10 9, SW11 0, SW12 -, SW13 =, SW14 BACKSPACE, SW15 ESCAPE, SW16 TAB, SW17 RESET, SW18 Q, SW19 W, SW2 1, SW20 E, SW21 R, SW22 T, SW23 Y, SW24 U, SW25 I, SW26 O, SW27 P, SW28 [, SW29 ], SW3 2, SW30 \, SW31 INSERT, SW32 CAPS LOCK, SW33 A, SW34 S, SW35 D, SW36 F, SW37 G, SW38 H, SW39 J, SW4 3, SW40 K, SW41 L, SW42 SHIFT, SW43 ;, SW44 ', SW45 ENTER, SW46 DELETE, SW47 Z, SW48 X, SW49 C, SW5 4, SW50 SHIFT, SW51 V, SW52 B, SW53 N, SW54 M, SW55 ,, SW56 ., SW57 /, SW58 UP ARROW, SW59 CTRL, SW6 5, SW60 ALT, SW61 MENU, SW62 SPACE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

Commit message: ACE Board Rev 1.1: name the ACIA as the R6551AP
U4's value field names the part tested on the AC6502 machines, the
R6551AP, where it said only "65C51". It changes in the schematic and on
the PCB, where the value sits on the silkscreen inside U4's socket
outline. The README's feature list and BOM say the same, and the
schematic PDF is plotted again. Rev 1.1 is unproduced; its production
files are regenerated with P1.7's 1N5819.

Rev 1.0 was fabricated and keeps "65C51". So the checker's parts table
now takes a value per revision (a config's `values`), and passes for
both revisions.

Co-Authored-By: Claude Opus 5.5 <noreply@anthropic.com>
Parts:
- U4: value 65C51 -> R6551AP
Changed lines of the file:
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@@
 			)
 		)
-		(property "Value" "65C51"
+		(property "Value" "R6551AP"
 			(at 7.62 35.25 0)
 			(layer "F.SilkS")
