File: Hardware/ACE Board/Rev 1.1/ACE Board.kicad_pcb (KiCad board)
At the start: 2 copper layers, 335 x 250 mm, 205 parts, among them J1 CTS EN, J10 AUDIO L, J11 DB9 MALE (DTE), J12 PS/2, J13 KEYBOARD, J14 AUDIO R, J15 AUDIO, J16 5V DC, J17 CART, J18 BUS, J19 VCC, J2 RESET SW, J20 POWER LED, J21 STORAGE, J3 DCD EN, J4 VDD, J5 JOYSTICK A, J6 PADDLES, J7 JOYSTICK B, J8 PORT B, J9 PORT A, SW1 `, SW10 9, SW11 0, SW12 -, SW13 =, SW14 BACKSPACE, SW15 ESCAPE, SW16 TAB, SW17 RESET, SW18 Q, SW19 W, SW2 1, SW20 E, SW21 R, SW22 T, SW23 Y, SW24 U, SW25 I, SW26 O, SW27 P, SW28 [, SW29 ], SW3 2, SW30 \, SW31 INSERT, SW32 CAPS LOCK, SW33 A, SW34 S, SW35 D, SW36 F, SW37 G, SW38 H, SW39 J, SW4 3, SW40 K, SW41 L, SW42 SHIFT, SW43 ;, SW44 ', SW45 ENTER, SW46 DELETE, SW47 Z, SW48 X, SW49 C, SW5 4, SW50 SHIFT, SW51 V, SW52 B, SW53 N, SW54 M, SW55 ,, SW56 ., SW57 /, SW58 UP ARROW, SW59 CTRL, SW6 5, SW60 ALT, SW61 MENU, SW62 SPACE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

Commit message: ACE Board Rev 1.1: reverse-polarity protection on the barrel jack
D5, a 1N5819 (DO-41), in series between the barrel jack (J16) and the
power switch (SW69), anode at the jack: the same part and place as on the
KIM Board. Rev 1.1 has not been produced, so the fix goes into it.

The netlist differs from before only there: J16 pin 1 -> D5 -> SW69 pin 2.
ERC and DRC are clean, nothing is unconnected, and check-schematics.mjs
passes. The production files, schematic PDF, renders and STEP model are
regenerated. The remaining silkscreen clearance warnings, which predate
this change, are excluded in the project.

The diode drops about 0.3-0.4 V, so VCC sits near 4.6 V; measure it under
full load on the first board built.

Co-Authored-By: Claude Opus 5.5 <noreply@anthropic.com>
Parts:
- added D5: 1N5819, Diode_THT:D_DO-41_SOD81_P10.16mm_Horizontal, F.Cu at (102.5, 91.3)
Connections:
- J16 pad 1: Net-(SW69-B) -> Net-(D5-A)
- SW69 pad 2: Net-(SW69-B) -> Net-(D5-K)
Routing:
- net Net-(D5-K): track 0.00 -> 17.3 mm
- net Net-(SW69-B): track 16.0 -> 0.00 mm
- net Net-(D5-A): track 0.00 -> 9.37 mm
